File: thermal-pcb/thermal-pcb.sch (KiCad schematic (older format))
At the start: 6 parts, among them J1 RS/E pins, J2 Conn_01x16_Female, J3 Data and power pins, J4 Temp sensor pins

Commit message: Update PCB scheme.
Parts:
- added J5: Switch RW, Connector_PinHeader_2.54mm:PinHeader_1x03_P2.54mm_Horizontal, symbol Connector:Conn_01x03_Male
- J1: footprint Connector_PinHeader_2.54mm:PinHeader_1x02_P2.54mm_Horizontal -> Connector_PinHeader_2.54mm:PinHeader_1x03_P2.54mm_Horizontal; symbol Connector:Conn_01x02_Male -> Connector:Conn_01x03_Male
Connections:
- net GND: now also J5.3 (Pin_3); no longer J2.5 (Pin_5)
- net at J2.6 (Pin_6): now also J1.3 (Pin_3); no longer J1.2 (Pin_2)
- new net: J2.5 (Pin_5), J5.2 (Pin_2)
- new net: J1.2 (Pin_2), J5.1 (Pin_1)
Changed lines of the file:
@@
 $EndDescr
-Wire Wire Line
-	3900 2900 5550 2900
-Connection ~ 5550 2900
 Wire Wire Line
 	3750 3050 3900 3050
@@
 Connection ~ 5550 3400
 Wire Wire Line
-	5550 3400 5550 2900
-Wire Wire Line
 	4200 3700 5400 3700
 Wire Wire Line
@@
 	5200 2200 5200 2100
 Wire Wire Line
-	5550 2200 5550 2900
+	5550 2200 5550 2700
 Wire Wire Line
 	5400 2300 5100 2300
@@
 Wire Wire Line
 	3750 2550 3750 3050
-Wire Wire Line
-	3900 2600 4100 2600
-Wire Wire Line
-	4100 2600 4100 2100
-Wire Wire Line
-	3900 2600 3900 2900
 Wire Wire Line
 	4200 2650 4200 2100
@@
 $EndComp
 $Comp
-L Connector:Conn_01x02_Male J1
+L Connector:Conn_01x03_Male J1
 U 1 1 5FD5DC3D
-P 3900 4750
-F 0 "J1" V 3962 4794 50  0000 L CNN
-F 1 "RS/E pins" V 4053 4794 50  0000 L CNN
-F 2 "Connector_PinHeader_2.54mm:PinHeader_1x02_P2.54mm_Horizontal" H 3900 4750 50  0001 C CNN
-F 3 "~" H 3900 4750 50  0001 C CNN
-	1    3900 4750
+P 4000 4750
+F 0 "J1" V 4062 4794 50  0000 L CNN
+F 1 "RS/E pins" V 4153 4794 50  0000 L CNN
+F 2 "Connector_PinHeader_2.54mm:PinHeader_1x03_P2.54mm_Horizontal" H 4000 4750 50  0001 C CNN
+F 3 "~" H 4000 4750 50  0001 C CNN
+	1    4000 4750
 	0    -1   -1   0
 $EndComp
@@
 	3900 3050 3900 4550
 Wire Wire Line
-	4050 2650 4050 4300
-Wire Wire Line
-	4050 4300 4000 4300
-Wire Wire Line
-	4000 4300 4000 4550
-Wire Wire Line
 	4800 4800 4900 4800
 Wire Wire Line
@@
 	6150 4150 6150 4650
 $Comp
-L power:+5V #PWR?
+L power:+5V #PWR0101
 U 1 1 5FCC39E4
 P 7000 4500
-F 0 "#PWR?" H 7000 4350 50  0001 C CNN
+F 0 "#PWR0101" H 7000 4350 50  0001 C CNN
 F 1 "+5V" H 7015 4673 50  0000 C CNN
 F 2 "" H 7000 4500 50  0001 C CNN
@@
 $EndComp
 $Comp
-L power:GND #PWR?
+L power:GND #PWR0102
 U 1 1 5FCC404B
 P 7400 4500
-F 0 "#PWR?" H 7400 4250 50  0001 C CNN
+F 0 "#PWR0102" H 7400 4250 50  0001 C CNN
 F 1 "GND" H 7405 4327 50  0000 C CNN
 F 2 "" H 7400 4500 50  0001 C CNN
@@
 $EndComp
 $Comp
-L power:PWR_FLAG #FLG?
+L power:PWR_FLAG #FLG0101
 U 1 1 5FCCD57C
 P 7000 4300
-F 0 "#FLG?" H 7000 4375 50  0001 C CNN
+F 0 "#FLG0101" H 7000 4375 50  0001 C CNN
 F 1 "PWR_FLAG" H 7000 4473 50  0000 C CNN
 F 2 "" H 7000 4300 50  0001 C CNN
@@
 $EndComp
 $Comp
-L power:PWR_FLAG #FLG?
+L power:PWR_FLAG #FLG0102
 U 1 1 5FCCDADC
 P 7400 4300
-F 0 "#FLG?" H 7400 4375 50  0001 C CNN
+F 0 "#FLG0102" H 7400 4375 50  0001 C CNN
 F 1 "PWR_FLAG" H 7400 4473 50  0000 C CNN
 F 2 "" H 7400 4300 50  0001 C CNN
@@
 	7000 4300 7000 4500
 $Comp
-L power:GND #PWR?
+L power:GND #PWR0103
 U 1 1 5FCD9462
 P 5550 5400
-F 0 "#PWR?" H 5550 5150 50  0001 C CNN
+F 0 "#PWR0103" H 5550 5150 50  0001 C CNN
 F 1 "GND" H 5555 5227 50  0000 C CNN
 F 2 "" H 5550 5400 50  0001 C CNN
@@
 	5400 4450 5400 4600
 $Comp
-L power:+5V #PWR?
+L power:+5V #PWR0104
 U 1 1 5FCE509D
 P 5800 5400
-F 0 "#PWR?" H 5800 5250 50  0001 C CNN
+F 0 "#PWR0104" H 5800 5250 50  0001 C CNN
 F 1 "+5V" H 5815 5573 50  0000 C CNN
 F 2 "" H 5800 5400 50  0001 C CNN
@@
 	-1   0    0    1
 $EndComp
+Wire Wire Line
+	4050 2650 4050 4300
+Wire Wire Line
+	4050 4300 4100 4300
+Wire Wire Line
+	4100 4300 4100 4550
+$Comp
+L Connector:Conn_01x03_Male J5
+U 1 1 5FD60558
+P 2850 2900
+F 0 "J5" V 2912 3044 50  0000 L CNN
+F 1 "Switch RW" V 3003 3044 50  0000 L CNN
+F 2 "Connector_PinHeader_2.54mm:PinHeader_1x03_P2.54mm_Horizontal" H 2850 2900 50  0001 C CNN
+F 3 "~" H 2850 2900 50  0001 C CNN
+	1    2850 2900
+	0    -1   -1   0
+$EndComp
+Wire Wire Line
+	4100 2100 4100 2150
+Wire Wire Line
+	4100 2150 2850 2150
+Wire Wire Line
+	2850 2150 2850 2700
+Wire Wire Line
+	2950 2700 5550 2700
+Connection ~ 5550 2700
+Wire Wire Line
+	2750 2700 2750 2550
+Wire Wire Line
+	2750 2550 3100 2550
+Wire Wire Line
+	3100 2550 3100 4200
+Wire Wire Line
+	3100 4200 4000 4200
+Wire Wire Line
+	4000 4200 4000 4550
+Wire Wire Line
+	5550 2700 5550 3400
 $EndSCHEMATC
