File: thermal-pcb/thermal-pcb.kicad_pcb (KiCad board)
At the start: 2 copper layers, 11 parts, among them J1 RS/E pins, J2 Conn_01x16_Female, J3 Data and power pins, J4 Temp sensor pins

Commit message: Update PCB scheme.
Parts:
- added J5: Switch RW, Connector_PinHeader_2.54mm:PinHeader_1x03_P2.54mm_Horizontal, F.Cu at (110.5, 63.0)
- J1: footprint Connector_PinHeader_2.54mm:PinHeader_1x02_P2.54mm_Horizontal -> Connector_PinHeader_2.54mm:PinHeader_1x03_P2.54mm_Horizontal
- moved 4.7k1 7.48 mm to (156.0, 65.0), turned to 270 degrees
- moved 10k1 5.49 mm to (129.5, 61.0)
- moved J1 2.59 mm to (120.7, 80.0)
Connections:
- 4.7k1 pad 1: Net-(4.7k1-Pad2) -> +5V
- 4.7k1 pad 2: +5V -> Net-(4.7k1-Pad2)
- J2 pad 4: Net-(J1-Pad2) -> Net-(J1-Pad1)
- J2 pad 5: GND -> Net-(J2-Pad5)
- J3 pad 3: Net-(J2-Pad14) -> Net-(J2-Pad13)
- J3 pad 4: Net-(J2-Pad13) -> Net-(J2-Pad14)
- J3 pad 6: Net-(J2-Pad11) -> GND
Routing:
- net +5V: track 144.7 -> 114.8 mm, vias 3 -> 1
- net Net-(J1-Pad1): track 0.00 -> 27.5 mm
- net Net-(J2-Pad5): track 0.00 -> 23.7 mm, vias 0 -> 1
- net Net-(10k1-Pad2): track 20.2 -> 15.4 mm
- net Net-(J1-Pad2): track 27.5 -> 22.9 mm
- net Net-(J1-Pad3): track 28.7 -> 27.6 mm

Commit message: Update PCB sheme (Stage I Complete)
Connections:
- J3 pad 3: Net-(J2-Pad13) -> Net-(J2-Pad14)
- J3 pad 4: Net-(J2-Pad14) -> Net-(J2-Pad13)
- J3 pad 6: GND -> Net-(J2-Pad11)
